Commit message: fixed package name in roslaunch

File: realsense2_camera/urdf/_d415.urdf.xacro (robot description, xacro)
@@ -46,5 +46,5 @@
         <geometry>
           <!-- <box size="${d415_cam_width} ${d415_cam_height} ${d415_cam_depth}"/> -->
-	         <mesh filename="package://realsense2_camera/meshes/d415.stl" />
+	         <mesh filename="package://realsense2_camera_alternate_1/meshes/d415.stl" />
         </geometry>
         <material name="aluminum"/>

File: realsense2_camera/urdf/_d435.urdf.xacro (robot description, xacro)
@@ -46,6 +46,6 @@
         <geometry>
           <!-- <box size="${d435_cam_width} ${d435_cam_height} ${d435_cam_depth}"/> -->
-	  <mesh filename="package://realsense2_camera/meshes/d435.dae" />
-          <!--<mesh filename="package://realsense2_camera/meshes/d435/d435.dae" />-->
+	  <mesh filename="package://realsense2_camera_alternate_1/meshes/d435.dae" />
+          <!--<mesh filename="package://realsense2_camera_alternate_1/meshes/d435/d435.dae" />-->
         </geometry>
         <material name="aluminum"/>

File: realsense2_camera/urdf/_r410.urdf.xacro (robot description, xacro)
@@ -39,5 +39,5 @@
         <geometry>
           <box size="${r410_cam_width} ${r410_cam_height} ${r410_cam_depth}"/>
-          <!--<mesh filename="package://realsense2_camera/meshes/r410/r410.dae" />-->
+          <!--<mesh filename="package://realsense2_camera_alternate_1/meshes/r410/r410.dae" />-->
         </geometry>
         <material name="aluminum"/>

File: realsense2_camera/urdf/_r430.urdf.xacro (robot description, xacro)
@@ -40,5 +40,5 @@
         <geometry>
           <box size="${r430_cam_width} ${r430_cam_height} ${r430_cam_depth}"/>
-          <!--<mesh filename="package://realsense2_camera/meshes/r430/r430.dae" />-->
+          <!--<mesh filename="package://realsense2_camera_alternate_1/meshes/r430/r430.dae" />-->
         </geometry>
         <material name="aluminum"/>

File: realsense2_camera/urdf/test_d415_camera.urdf.xacro (robot description, xacro)
@@ -1,5 +1,5 @@
 <?xml version="1.0"?>
 <robot name="realsense2_camera" xmlns:xacro="http://ros.org/wiki/xacro">
-  <xacro:include filename="$(find realsense2_camera)/urdf/_d415.urdf.xacro"/>
+  <xacro:include filename="$(find realsense2_camera_alternate_1)/urdf/_d415.urdf.xacro"/>
   <link name="base_link" />
   <sensor_d415 parent="base_link">

File: realsense2_camera/urdf/test_d435_camera.urdf.xacro (robot description, xacro)
@@ -1,5 +1,5 @@
 <?xml version="1.0"?>
 <robot name="realsense2_camera" xmlns:xacro="http://ros.org/wiki/xacro">
-  <xacro:include filename="$(find realsense2_camera)/urdf/_d435.urdf.xacro"/>
+  <xacro:include filename="$(find realsense2_camera_alternate_1)/urdf/_d435.urdf.xacro"/>
   <link name="base_link" />
   <sensor_d435 parent="base_link">

File: realsense2_camera/urdf/test_r410_camera.urdf.xacro (robot description, xacro)
@@ -1,5 +1,5 @@
 <?xml version="1.0"?>
 <robot name="realsense2_camera" xmlns:xacro="http://ros.org/wiki/xacro">
-  <xacro:include filename="$(find realsense2_camera)/urdf/_r410.urdf.xacro"/>
+  <xacro:include filename="$(find realsense2_camera_alternate_1)/urdf/_r410.urdf.xacro"/>
   <link name="base_link" />
   <sensor_r410 parent="base_link">

File: realsense2_camera/urdf/test_r430_camera.urdf.xacro (robot description, xacro)
@@ -1,5 +1,5 @@
 <?xml version="1.0"?>
 <robot name="realsense2_camera" xmlns:xacro="http://ros.org/wiki/xacro">
-  <xacro:include filename="$(find realsense2_camera)/urdf/_r430.urdf.xacro"/>
+  <xacro:include filename="$(find realsense2_camera_alternate_1)/urdf/_r430.urdf.xacro"/>
   <link name="base_link" />
   <sensor_r430 parent="base_link">
